File: KiCad Files/Mixor-Image-v5.kicad_sch (KiCad schematic)
At the start: 51 parts, among them J1 Conn_01x03_Male, J2 Conn_01x03_Female, J3 Conn_01x03_Male, J4 Conn_01x03_Female, U1 TL072, U2 TL072

Commit message: adds C/D logo, change resistors to SMD
Parts:
- R2: footprint Resistor_THT:R_Axial_DIN0204_L3.6mm_D1.6mm_P1.90mm_Vertical -> PCM_Resistor_SMD_AKL:R_0201_0603Metric
Changed lines of the file:
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@@
 			)
 		)
-		(property "Footprint" "Resistor_THT:R_Axial_DIN0204_L3.6mm_D1.6mm_P1.90mm_Vertical"
+		(property "Footprint" "PCM_Resistor_SMD_AKL:R_0201_0603Metric"
 			(at 80.264 29.464 90)
 			(effects
