File: KiCad Files/PCBs/Mixor-Image-v5.kicad_pcb (KiCad board)
At the start: 2 copper layers, 60.6 x 46 mm, 80 parts, among them J1 Conn_01x03_Male, J2 Conn_01x03_Female, J3 Conn_01x03_Male, J4 Conn_01x03_Female, U1 TL072, U2 TL072

Commit message: version submitted to JLCPCB 2024-06-09
Connections:
- L-O1 pad T: Net-(J3-Pin_3) -> Net-(J3-Pin_1)
- R-O1 pad T: Net-(J3-Pin_1) -> Net-(J3-Pin_3)
- R10 pad 2: Net-(J1-Pin_3) -> Net-(J1-Pin_1)
- R11 pad 2: Net-(J1-Pin_1) -> Net-(J1-Pin_3)
- R12 pad 2: Net-(J1-Pin_3) -> Net-(J1-Pin_1)
- R13 pad 2: Net-(J1-Pin_1) -> Net-(J1-Pin_3)
- R14 pad 2: Net-(ST-IN1-Pin_3) -> Net-(ST-IN1-Pin_1)
- R15 pad 1: Net-(ST-IN1-Pin_1) -> Net-(ST-IN1-Pin_3)
- R2 pad 2: Net-(J1-Pin_3) -> Net-(J1-Pin_1)
- R3 pad 2: Net-(J1-Pin_1) -> Net-(J1-Pin_3)
- R4 pad 2: Net-(J1-Pin_3) -> Net-(J1-Pin_1)
- R5 pad 2: Net-(J1-Pin_1) -> Net-(J1-Pin_3)
- R6 pad 2: Net-(J1-Pin_3) -> Net-(J1-Pin_1)
- R7 pad 2: Net-(J1-Pin_1) -> Net-(J1-Pin_3)
- R8 pad 2: Net-(J1-Pin_3) -> Net-(J1-Pin_1)
- R9 pad 2: Net-(J1-Pin_1) -> Net-(J1-Pin_3)
- ST-OUT1 pad 1: Net-(J4-Pin_3) -> Net-(J4-Pin_1)
- ST-OUT1 pad 3: Net-(J4-Pin_1) -> Net-(J4-Pin_3)
Routing:
- net GND: track 0.00 -> 127.1 mm
- net Net-(J4-Pin_1): track 9.36 -> 47.5 mm, vias 0 -> 1
- net Net-(J1-Pin_3): track 83.0 -> 112.0 mm, vias 2 -> 0
- net Net-(C3-Pad2): track 20.9 -> 11.3 mm
- net Net-(R16-Pad2): track 20.5 -> 12.3 mm
- net Net-(J4-Pin_3): track 34.4 -> 40.8 mm
- net Net-(J1-Pin_1): track 89.0 -> 82.6 mm
- net Net-(J3-Pin_3): track 3.45 -> 9.72 mm
- net Net-(J3-Pin_1): track 3.45 -> 9.27 mm
- net Net-(ST-IN1-Pin_3): track 10.2 -> 6.55 mm
- net Net-(U2B--): track 26.2 -> 29.5 mm
- net Net-(J2-Pin_3): track 34.7 -> 31.9 mm
- net -12V: track 65.6 -> 68.1 mm
- net Net-(J2-Pin_1): track 16.5 -> 15.1 mm
- net Net-(C2-Pad2): track 14.3 -> 13.2 mm
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Other:
- board text added: "JLCJLCJLCJLC"
