File: KiCad Files/PCBs/Near-Mix-v5.kicad_sch (KiCad schematic)
At the start: 51 parts, among them J1 Conn_01x03_Male, J2 Conn_01x03_Female, J3 Conn_01x03_Male, J4 Conn_01x03_Female, U1 TL072, U2 TL072

Commit message: rename Kicad files and update schematic info
Other:
- company: Modular Maculata -> ${company}
- title: Mixor Image -> ${product}
Changed lines of the file:
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@@
 	(paper "A4")
 	(title_block
-		(title "Mixor Image")
-		(date "2022-03-31")
-		(rev "5")
-		(company "Modular Maculata")
-		(comment 1 "(inspired by nearness mixer)")
+		(title "${product}")
+		(date "2024-10-23")
+		(rev "6")
+		(company "${company}")
+		(comment 1 "(derived from mixor image, inspired by nearness mixer)")
 		(comment 2 "CONSTANT POWER PANNING (-35, -15, 0, 15, 35)")
 	)

Commit message: first fully SMD version ordered from JLCPCB 2024-10-24
Parts:
- C1: footprint Capacitor_THT:C_Rect_L4.0mm_W2.0mm_P4.00mm -> Capacitor_SMD:C_1206_3216Metric
- C2, C3: footprint Capacitor_THT:C_Disc_D4.0mm_W1.6mm_P3.0mm -> Capacitor_SMD:C_1206_3216Metric
- C4, C5: footprint Capacitor_THT:C_Radial_D5.0mm_H11.0mm_P2.00mm -> Capacitor_SMD:CP_Elec_3x5.3
- C6, C7, C8, C9: footprint Resistor_THT:R_Axial_DIN0204_L3.6mm_D1.6mm_P2.54mm_Vertical -> Capacitor_SMD:C_1206_3216Metric
- CEN1, CEN2, L-IN1, L-O1, R-IN1, R-IN2, R-O1: footprint AudioJacks:Jack_3.5mm_QingPu_WQP-PJ398SM_Vertical -> Audio Jacks:Jack_3.5mm_QingPu_WQP-PJ398SM_Vertical
- D1, D2: footprint Diode_THT:D_A-405_P2.54mm_Vertical_AnodeUp -> Diode_SMD:D_1206_3216Metric
- L_IN2: footprint thonk:Jack_3.5mm_QingPu_WQP-PJ301M-12_Vertical -> Audio Jacks:Jack_3.5mm_QingPu_WQP-PJ398SM_Vertical
- R1, R10, R11, R12, R13, R14, R15, R16, R17, R18, R19, R2, R20, R21, R22, R23, R3, R4, R5, R6, R7, R8, R9: footprint Resistor_THT:R_Axial_DIN0204_L3.6mm_D1.6mm_P1.90mm_Vertical -> PCM_4ms_Resistor:R_1206_3216Metric
- U1, U2: footprint Package_DIP:DIP-8_W7.62mm_Socket -> PCM_Package_SO_AKL:SOIC-8_3.9x4.9mm_P1.27mm
Connections:
- net CEN_IN_1_net: now reaches C1.1, CEN1.T
- no-connect marks 0 -> 2

Commit message: uses different footprint for diodes - JLC didn't have parts to match previous updates labels so they are oriented sanely and not cut off by pads ordered 2024-10-25 order for previous commit cancelled
Parts:
- D1, D2: footprint Diode_SMD:D_1206_3216Metric -> Diode_SMD:D_SOD-123F
Changed lines of the file:
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@@
 			)
 		)
-		(property "Footprint" "Diode_SMD:D_1206_3216Metric"
+		(property "Footprint" "Diode_SMD:D_SOD-123F"
 			(at 218.44 157.48 0)
 			(effects
@@
 			)
 		)
-		(property "Footprint" "Diode_SMD:D_1206_3216Metric"
+		(property "Footprint" "Diode_SMD:D_SOD-123F"
 			(at 218.44 139.7 0)
 			(effects
