File: KiCad Files/panel/Mixor_Image-Plain_Panel.kicad_pcb (KiCad board)
At the start: 2 copper layers, 60.6 x 39.6 mm, 39 parts

Commit message: version submitted to JLCPCB 2024-06-09
Parts:
- moved ? 142.3 mm to (141.7, 117.1) (x4)
- moved ? 142.3 mm to (126.9, 115.2) (x2)
- moved ? 142.3 mm to (135.7, 89.8) (x3)
- moved ? 142.3 mm to (150.8, 116.3) (x3)
- moved ? 142.3 mm to (151.0, 115.7)
- moved ? 142.3 mm to (123.9, 90.9)
- moved ? 142.3 mm to (142.0, 117.1)
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Other:
- board size 60.6 x 39.6 mm -> 60.6 x 39.7 mm
- board text added: "JLCJLCJLCJLC"

Commit message: first fully SMD version ordered from JLCPCB 2024-10-24
Parts:
- removed the ? at (142.0, 117.1)
Other:
- board text removed: "A NEAR MIX"
- board text removed: "COMMON DENOMINATOR DEVICES “A NEAR MIX” PANEL v1 2024"
